File: kicad/nice_pillz_niceview_v9.kicad_pcb (KiCad board)
At the start: 2 copper layers, 100 x 86 mm, 27 parts, among them J1 Conn_01x13, J2 Conn_01x13, J3 Conn_01x13, J4 Conn_01x13, J5 Conn_01x10, J6 Conn_01x10, J7 Conn_01x13, J8 Conn_01x13, M1 MountingHole_6.4mm_M6, M3 MountingHole_4.3mm_M4, M4 MountingHole_4.3mm_M4, U1 nice!nanov2, U2 74HC595

Commit message: New board
Parts:
- added J9: NiceView, Local:NiceView_1x05_P2.54mm_V, F.Cu at (160.0, 73.4)
- moved G*** 61.5 mm to (113.8, 66.0), turned to 0 degrees
Connections:
- Battery pad 2: BAT- -> GND
- R1 pad 2: /LED_CAPS_LOCK -> /PWR_LED
- U2 pad 15: (no net) -> /PWR_LED
Routing:
- net /SPI_MOSI: track 31.0 -> 123.3 mm, vias 0 -> 3
- net /SPI_SCK: track 41.3 -> 118.9 mm, vias 2 -> 4
- net GND: track 10.8 -> 66.9 mm
- net /PWR_LED: track 0.00 -> 55.1 mm, vias 0 -> 2
- net BAT-: track 43.5 -> 0.00 mm
- net /LED_CAPS_LOCK: track 47.4 -> 90.1 mm, vias 1 -> 2
- net +5V: track 33.2 -> 55.0 mm, vias 0 -> 1
- net /ROW_3: track 76.3 -> 73.7 mm
- net /ROW_5: track 69.5 -> 68.0 mm
- net /ROW_11: track 65.8 -> 64.9 mm
- net /ROW_8: track 111.2 -> 110.3 mm
Other:
- board text added: "Nice Pillz View github.com/a10kiloham/nicepillzview v1.0 29 Aug 2026 (built from github/nol00p/nicepillz)"
